File: COM_PCB.kicad_sch (KiCad schematic)
At the start: 0 parts

Commit message: KiCad 0.3v
Improved aesthetics.
Other:
- sheet SI4463: file file5FC06DBC.kicad_sch -> UHF.kicad_sch

Commit message: 0.1v COM_PCB KiCad
First iteration of COM PCB.
Other:
- sheet GPRS ports: added none; removed GSM_CTS, GSM_RTS
- sheet IO ports: added SW_CLK, SW_IO, ~{RST}; removed RX
- sheet MCU ports: added DEBUG_TX, SW_CLK, SW_IO, ~{RST}; removed GSM_CTS, GSM_RTS, RF_DIO1, RX, TX
- sheet SI4463 ports: added none; removed GPIO1

Commit message: V1
Other:
- company: (none) -> BASEMENT
Changed lines of the file:
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@@
 (kicad_sch (version 20211123) (generator eeschema)
   (paper "A4")
+  (title_block
+    (date "%%date%%")
+    (rev "%%version%%")
+    (company "BASEMENT")
+  )
   (junction (at 161.29 63.5) (diameter 0) (color 0 0 0 0)
   )
