File: IO.kicad_sch (KiCad schematic)
At the start: 2 parts, among them J5 Conn_01x08_Male, J6 02x12

Commit message: KiCad 0.2v
Schematics done.
Have to assign footprints to corresponding components.
Completely rework PCB.
Parts:
- removed J5: Conn_01x08_Male, symbol Connector:Conn_01x08_Male
- removed J6: 02x12, LOCAL:SAMTEC-SSW-112-02-X-D-RA, symbol Connector_Generic:Conn_02x12_Top_Bottom
- added J5: 02x12, LOCAL:SAMTEC-SSW-112-02-X-D-RA, symbol Connector_Generic:Conn_02x12_Top_Bottom
- added J6: DEBUG_INTERFACE_L, symbol Connector:Conn_01x08_Male
- added J7: DEBUG_INTERFACE_R, symbol Connector:Conn_01x08_Male
Connections:
- net GND: now also J5.1 (Pin_1), J5.12 (Pin_12), J5.13 (Pin_13), J5.24 (Pin_24), J6.1 (Pin_1), J6.8 (Pin_8), J7.1 (Pin_1), J7.8 (Pin_8)
- net MCU_RX: now also J5.19 (Pin_19), J5.6 (Pin_6)
- net MCU_TX: now also J5.18 (Pin_18), J5.7 (Pin_7)
- net RX: now also J6.4 (Pin_4)
- net TX: now also J6.3 (Pin_3)
- new net +3V3: J5.11 (Pin_11), J5.14 (Pin_14), J6.7 (Pin_7)
- new net +4V: J5.2 (Pin_2), J5.23 (Pin_23), J6.2 (Pin_2)
- new net GPS_RX: J6.6 (Pin_6)
- new net GPS_TX: J6.5 (Pin_5)
- new net GSM_RX: J7.6 (Pin_6)
- new net GSM_TX: J7.7 (Pin_7)
- new net RF_MISO: J7.4 (Pin_4)
- new net RF_MOSI: J7.3 (Pin_3)
- new net RF_NSS: J7.5 (Pin_5)
- new net RF_SCK: J7.2 (Pin_2)
- no-connect marks 18 -> 12

Commit message: KiCad 0.3v
Improved aesthetics.
Parts:
- removed J5: 02x12, LOCAL:SAMTEC-SSW-112-02-X-D-RA, symbol Connector_Generic:Conn_02x12_Top_Bottom
- removed J6: DEBUG_INTERFACE_L, symbol Connector:Conn_01x08_Male
- removed J7: DEBUG_INTERFACE_R, symbol Connector:Conn_01x08_Male
- added J5: Conn_02x10_Top_Bottom, Connector_PinHeader_2.54mm:PinHeader_2x20_P2.54mm_Horizontal, symbol Connector_Generic:Conn_02x10_Top_Bottom
- added J6: Conn_01x14_Male, Connector_PinHeader_2.54mm:PinHeader_1x14_P2.54mm_Horizontal, symbol Connector:Conn_01x14_Male
Connections:
- net +3V3: now also J5.12 (Pin_12), J5.9 (Pin_9), J6.13 (Pin_13)
- net +4V: now also J5.19 (Pin_19), J5.2 (Pin_2), J6.2 (Pin_2)
- net GND: now also J5.1 (Pin_1), J5.10 (Pin_10), J5.11 (Pin_11), J5.20 (Pin_20), J6.1 (Pin_1), J6.14 (Pin_14)
- net GPS_RX: now also J6.6 (Pin_6)
- net GPS_TX: now also J6.5 (Pin_5)
- net GSM_RX: now also J6.11 (Pin_11)
- net GSM_TX: now also J6.12 (Pin_12)
- net MCU_RX: now also J5.16 (Pin_16), J5.5 (Pin_5)
- net MCU_TX: now also J5.15 (Pin_15), J5.6 (Pin_6)
- net RF_MISO: now also J6.9 (Pin_9)
- net RF_MOSI: now also J6.8 (Pin_8)
- net RF_NSS: now also J6.10 (Pin_10)
- net RF_SCK: now also J6.7 (Pin_7)
- net RX: now also J6.4 (Pin_4)
- net TX: now also J6.3 (Pin_3)
- no-connect marks 12 -> 8
Other:
- note added: "Backbone connector"
- note added: "Debug interface"
- note added: "Power flags"

Commit message: 0.1v COM_PCB KiCad
First iteration of COM PCB.
Parts:
- removed J5: Conn_02x10_Top_Bottom, Connector_PinHeader_2.54mm:PinHeader_2x20_P2.54mm_Horizontal, symbol Connector_Generic:Conn_02x10_Top_Bottom
- removed J6: Conn_01x14_Male, Connector_PinHeader_2.54mm:PinHeader_1x14_P2.54mm_Horizontal, symbol Connector:Conn_01x14_Male
- added H1, H2: Spacer, MountingHole:MountingHole_3.2mm_M3, symbol Mechanical:MountingHole
- added J5: BackBone, Connector_PinSocket_2.54mm:PinSocket_2x10_P2.54mm_Horizontal, symbol Connector_Generic:Conn_02x10_Odd_Even
- added J6: D1, Connector_PinSocket_2.54mm:PinSocket_1x08_P2.54mm_Horizontal, symbol Connector_Generic:Conn_01x08
- added J7: D2, Connector_PinSocket_2.54mm:PinSocket_1x08_P2.54mm_Horizontal, symbol Connector_Generic:Conn_01x08
Connections:
- net +3V3: now also J5.17 (Pin_17), J5.18 (Pin_18), J7.7 (Pin_7)
- net +4V: now also J5.3 (Pin_3), J5.4 (Pin_4), J6.6 (Pin_6)
- net GND: now also J5.1 (Pin_1), J5.19 (Pin_19), J5.2 (Pin_2), J5.20 (Pin_20), J6.1 (Pin_1), J7.8 (Pin_8)
- net GPS_RX: now also J7.1 (Pin_1)
- net GPS_TX: now also J7.2 (Pin_2)
- net GSM_RX: now also J6.7 (Pin_7)
- net GSM_TX: now also J6.8 (Pin_8)
- net MCU_RX: now also J5.11 (Pin_11), J5.12 (Pin_12)
- net MCU_TX: now also J5.10 (Pin_10), J5.9 (Pin_9)
- net RF_MISO: now also J7.5 (Pin_5)
- net RF_MOSI: now also J7.4 (Pin_4)
- net RF_NSS: now also J7.3 (Pin_3)
- net RF_SCK: now also J7.6 (Pin_6)
- net TX: now also J6.5 (Pin_5)
- new net SW_CLK: J6.4 (Pin_4)
- new net SW_IO: J6.3 (Pin_3)
- new net ~{RST}: J6.2 (Pin_2)
Other:
- note added: "BACKBONE_CONN"
- note added: "DEBUG_CONN"
- note added: "INTERCONNECT_HOLDERS"
- note removed: "Backbone connector"
- note removed: "Debug interface"

Commit message: V1
Other:
- company: (none) -> BASEMENT
- title: (none) -> I/O
Changed lines of the file:
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@@
 (kicad_sch (version 20211123) (generator eeschema)
   (paper "A4")
+  (title_block
+    (title "I/O")
+    (date "%%date%%")
+    (rev "%%version%%")
+    (company "BASEMENT")
+  )
   (junction (at 44.5516 32.6136) (diameter 0) (color 0 0 0 0)
   )
