File: UHF.kicad_sch (KiCad schematic)
At the start: 29 parts, among them J1 SMA, U1 SI4463, U2 AS179-92LF, X1 TCXO 30 MHz

Commit message: 0.1v COM_PCB KiCad
First iteration of COM PCB.
Parts:
- added J8: BMI-S-205-C, RF_Shielding:Laird_Technologies_BMI-S-205-F_38.10x25.40mm, symbol Device:RFShield_OnePiece
- U1: footprint (none) -> Package_DFN_QFN:QFN-20-1EP_4x4mm_P0.5mm_EP2.6x2.6mm_ThermalVias
Connections:
- net GND: now also J8.1 (Shield)
- net GPIO1: no longer names the net of U1.10 (GPIO1)
- no-connect marks 3 -> 4
Changed lines of the file:
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@@
   )
   (no_connect (at 82.931 41.783))
+  (no_connect (at 88.265 57.023))
   (no_connect (at 62.611 46.863))
   (no_connect (at 114.3 38.608))
@@
     (effects (font (size 1.27 1.27)) (justify right))
   )
-  (hierarchical_label "GPIO1" (shape input) (at 88.265 57.023 0)
-    (effects (font (size 1.27 1.27)) (justify left))
-  )
   (hierarchical_label "GPIO0" (shape input) (at 88.265 54.483 0)
     (effects (font (size 1.27 1.27)) (justify left))
@@
     (pin "1")
   )
+  (symbol (lib_id "Device:RFShield_OnePiece") (at 218.44 91.44 0) (unit 1)
+    (in_bom yes) (on_board yes) (fields_autoplaced)
+    (property "Reference" "J8" (id 0) (at 234.95 90.1699 0)
+      (effects (font (size 1.27 1.27)) (justify left))
+    )
+    (property "Value" "BMI-S-205-C" (id 1) (at 234.95 92.7099 0)
+      (effects (font (size 1.27 1.27)) (justify left))
+    )
+    (property "Footprint" "RF_Shielding:Laird_Technologies_BMI-S-205-F_38.10x25.40mm" (id 2) (at 218.44 93.98 0)
+      (effects (font (size 1.27 1.27)) hide)
+    )
+    (property "Datasheet" "~" (id 3) (at 218.44 93.98 0)
+      (effects (font (size 1.27 1.27)) hide)
+    )
+    (pin "1")
+  )
   (symbol (lib_id "Device:C_Small") (at 202.946 29.718 90) (unit 1)
     (in_bom yes) (on_board yes)
@@
     (pin "1")
     (pin "2")
+  )
+  (symbol (lib_id "power:GND") (at 218.44 101.6 0) (unit 1)
+    (in_bom yes) (on_board yes) (fields_autoplaced)
+    (property "Reference" "#PWR0136" (id 0) (at 218.44 107.95 0)
+      (effects (font (size 1.27 1.27)) hide)
+    )
+    (property "Value" "GND" (id 1) (at 218.44 106.68 0))
+    (property "Footprint" "" (id 2) (at 218.44 101.6 0)
+      (effects (font (size 1.27 1.27)) hide)
+    )
+    (property "Datasheet" "" (id 3) (at 218.44 101.6 0)
+      (effects (font (size 1.27 1.27)) hide)
+    )
+    (pin "1")
   )
   (symbol (lib_id "Device:C_Small") (at 185.42 91.948 270) (unit 1)
@@
     (property "Reference" "U1" (id 0) (at 63.881 30.353 0))
     (property "Value" "SI4463" (id 1) (at 66.421 32.893 0))
-    (property "Footprint" "" (id 2) (at 72.771 18.923 0)
-      (effects (font (size 1.27 1.27)) hide)
-    )
+    (property "Footprint" "Package_DFN_QFN:QFN-20-1EP_4x4mm_P0.5mm_EP2.6x2.6mm_ThermalVias" (id 2) (at 72.771 18.923 0)
+      (effects (font (size 1.27 1.27)) hide)
+    )

Commit message: solved issues
Crystal changes and some routing.
Parts:
- X1: footprint Crystal:Crystal_SMD_2016-4Pin_2.0x1.6mm -> Crystal:Crystal_SMD_2520-4Pin_2.5x2.0mm
Changed lines of the file:
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@@
       (effects (font (size 1.27 1.27)) (justify left))
     )
-    (property "Footprint" "Crystal:Crystal_SMD_2016-4Pin_2.0x1.6mm" (id 2) (at 149.86 47.498 0)
+    (property "Footprint" "Crystal:Crystal_SMD_2520-4Pin_2.5x2.0mm" (id 2) (at 149.86 47.498 0)
       (effects (font (size 1.27 1.27)) hide)
     )

Commit message: V1
Other:
- company: (none) -> BASEMENT
- title: (none) -> Transceiver SI4463
Changed lines of the file:
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@@
 (kicad_sch (version 20211123) (generator eeschema)
   (paper "A4")
+  (title_block
+    (title "Transceiver SI4463")
+    (date "%%date%%")
+    (rev "%%version%%")
+    (company "BASEMENT")
+  )
   (junction (at 246.38 32.258) (diameter 0) (color 0 0 0 0)
   )
