File: gprs.kicad_sch (KiCad schematic)
At the start: 8 parts, among them J1 Conn_Coaxial, J2 SIM_Card

Commit message: KiCad 0.2v
Schematics done.
Have to assign footprints to corresponding components.
Completely rework PCB.
Parts:
- removed C1, C3: 0.1uF, Capacitor_SMD:C_0603_1608Metric, symbol Device:C_Small
- removed C11, C2: 220uF, Capacitor_Tantalum_SMD:CP_EIA-3216-10_Kemet-I_Pad1.58x1.35mm_HandSolder, symbol Device:C_Small
- removed J1: Conn_Coaxial, Connector_Coaxial:SMA_Amphenol_132134-16_Vertical, symbol Connector:Conn_Coaxial
- removed J2: SIM_Card, footprints:MOLEX_78800-0001, symbol Connector:SIM_Card
- removed R1: 10k, Capacitor_SMD:C_0603_1608Metric, symbol Device:R_Small
- added C20, C22: 220uF, Capacitor_Tantalum_SMD:CP_EIA-3216-10_Kemet-I_Pad1.58x1.35mm_HandSolder, symbol Device:C_Small
- added C21, C23: 0.1uF, Capacitor_SMD:C_0603_1608Metric, symbol Device:C_Small
- added J3: Conn_Coaxial, Connector_Coaxial:SMA_Amphenol_132134-16_Vertical, symbol Connector:Conn_Coaxial
- added J4: SIM_Card, footprints:MOLEX_78800-0001, symbol Connector:SIM_Card
- added R4: 10k, Capacitor_SMD:C_0603_1608Metric, symbol Device:R_Small
Connections:
- net ANT: now also J3.1 (In)
- net GND: now also C20.2, C21.2, C22.2, C23.2, J3.2 (Ext), J4.5 (GND)
- net GSM_RST: now also C21.1, R4.2
- net SIM_CLK: now also J4.3 (CLK)
- net SIM_DATA: now also J4.7 (I/O)
- net SIM_RST: now also J4.2 (RST)
- net SIM_VSIM: now also J4.1 (VCC)
- net 4V renamed +4V
- net +4V: now also C20.1, C22.1, C23.1, R4.1

Commit message: KiCad 0.3v
Improved aesthetics.
Parts:
- GSM1: symbol test:A6_GSM -> schematics:A6_GSM
- J3: value Conn_Coaxial -> SMA
- J4: value SIM_Card -> Card_Holder
- R4: value 10k -> 12k
Other:
- note added: "Antena connector"
- note added: "Decoupling capacitors"
- note added: "GSM A6 module"
- note added: "Reset"
- note added: "Sim card holder"
- note added: "Use tantalum for decoupling"
- note removed: "Use tantalum for 470uF smaller"
- moved on the sheet: C21, C22, C23, GSM1, J3, J4, R4

Commit message: 0.1v COM_PCB KiCad
First iteration of COM PCB.
Parts:
- C20, C22: footprint Capacitor_Tantalum_SMD:CP_EIA-3216-10_Kemet-I_Pad1.58x1.35mm_HandSolder -> Capacitor_Tantalum_SMD:CP_EIA-3528-21_Kemet-B
- GSM1: footprint MODULE -> footprints:A6_GSM
Connections:
- net GSM_CTS: no longer names the net of GSM1.10 (UART_CTS/GPIO5)
- net GSM_RTS: no longer names the net of GSM1.11 (UART_RTS/GPIO7)
- no-connect marks 20 -> 22
Changed lines of the file:
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@@
   (no_connect (at 90.17 50.546))
   (no_connect (at 36.83 42.926))
+  (no_connect (at 36.83 50.546))
   (no_connect (at 90.17 60.706))
   (no_connect (at 90.17 40.386))
@@
   (no_connect (at 36.83 35.306))
   (no_connect (at 36.83 40.386))
+  (no_connect (at 36.83 53.086))
   (no_connect (at 36.83 68.326))
   (no_connect (at 90.17 58.166))
@@
     (stroke (width 0) (type default) (color 0 0 0 0))
   )
-  (wire (pts (xy 34.29 50.546) (xy 36.83 50.546))
-    (stroke (width 0) (type default) (color 0 0 0 0))
-  )
   (polyline (pts (xy 133.0452 70.6628) (xy 133.0452 42.2148))
     (stroke (width 0) (type default) (color 0 0 0 0))
@@
   )
   (polyline (pts (xy 168.91 42.2148) (xy 135.636 42.2148))
-    (stroke (width 0) (type default) (color 0 0 0 0))
-  )
-  (wire (pts (xy 36.83 53.086) (xy 34.29 53.086))
     (stroke (width 0) (type default) (color 0 0 0 0))
   )
@@
   (label "SIM_DATA" (at 147.6756 35.7632 0)
     (effects (font (size 1.27 1.27)) (justify left bottom))
-  )
-  (hierarchical_label "GSM_CTS" (shape input) (at 34.29 50.546 180)
-    (effects (font (size 1.27 1.27)) (justify right))
-  )
-  (hierarchical_label "GSM_RTS" (shape input) (at 34.29 53.086 180)
-    (effects (font (size 1.27 1.27)) (justify right))
   )
   (hierarchical_label "GSM_RST" (shape input) (at 118.0592 56.4388 180)
@@
       (effects (font (size 1.27 1.27)) (justify left))
     )
-    (property "Footprint" "Capacitor_Tantalum_SMD:CP_EIA-3216-10_Kemet-I_Pad1.58x1.35mm_HandSolder" (id 2) (at 113.4364 28.8544 0)
+    (property "Footprint" "Capacitor_Tantalum_SMD:CP_EIA-3528-21_Kemet-B" (id 2) (at 113.4364 28.8544 0)
       (effects (font (size 1.27 1.27)) hide)
     )
@@
       (effects (font (size 1.27 1.27)) (justify left))
     )
-    (property "Footprint" "Capacitor_Tantalum_SMD:CP_EIA-3216-10_Kemet-I_Pad1.58x1.35mm_HandSolder" (id 2) (at 122.3264 28.8544 0)
+    (property "Footprint" "Capacitor_Tantalum_SMD:CP_EIA-3528-21_Kemet-B" (id 2) (at 122.3264 28.8544 0)
       (effects (font (size 1.27 1.27)) hide)
     )
@@
   (symbol (lib_id "schematics:A6_GSM") (at 63.5 53.086 0) (unit 1)
     (in_bom yes) (on_board yes) (fields_autoplaced)
-    (property "Reference" "GSM1" (id 0) (at 63.5 18.034 0))
-    (property "Value" "A6_GSM" (id 1) (at 63.5 20.574 0))
-    (property "Footprint" "MODULE" (id 2) (at 63.5 81.026 0)
-      (effects (font (size 1.27 1.27)) hide)
-    )
+    (property "Reference" "GSM1" (id 0) (at 63.5 17.78 0))
+    (property "Value" "A6_GSM" (id 1) (at 63.5 20.32 0))
+    (property "Footprint" "footprints:A6_GSM" (id 2) (at 63.5 81.026 0)
+      (effects (font (size 1.27 1.27)) hide)
+    )

Commit message: V1
Other:
- company: (none) -> BASEMENT
- title: (none) -> GSM A6
Changed lines of the file:
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@@
 (kicad_sch (version 20211123) (generator eeschema)
   (paper "A4")
+  (title_block
+    (title "GSM A6")
+    (date "%%date%%")
+    (rev "%%version%%")
+    (company "BASEMENT")
+  )
   (junction (at 92.71 78.486) (diameter 0) (color 0 0 0 0)
   )
